File: PLC4UNI/untitled.kicad_sch (KiCad schematic)
At the start: 0 parts

Commit message: esquematico general, sin circuitos definidos
Parts:
- added R1: 2.2k, symbol Device:R
- added U1: ESP32-S3-WROOM-1, RF_Module:ESP32-S3-WROOM-1, symbol RF_Module:ESP32-S3-WROOM-1
Connections:
- new net +3.3V: R1.1, U1.2 (3V3)
- new net ACC_CS: U1.7 (IO7)
- new net CLK: U1.22 (IO14)
- new net CS: U1.19 (IO11)
- new net EMRX: U1.36 (RXD0)
- new net EM_1X: U1.37 (TXD0)
- new net EN: R1.2, U1.3 (EN)
- new net GND: U1.1 (GND), U1.40 (GND), U1.41 (GND)
- new net GPIO1: U1.8 (IO15)
- new net GPIO2: U1.9 (IO16)
- new net I2C_SCL: U1.11 (IO18)
- new net I2C_SDA: U1.10 (IO17)
- new net IN_NPN0: U1.27 (IO0)
- new net IN_NPN1: U1.39 (IO1)
- new net IN_NPN2: U1.38 (IO2)
- new net IN_NPN3: U1.15 (IO3)
- new net IN_PNP0: U1.4 (IO4)
- new net IN_PNP1: U1.5 (IO5)
- new net IN_VAC_ADS: U1.6 (IO6)
- new net LED_INFO: U1.23 (IO21)
- new net MISO: U1.20 (IO12)
- new net MOSI: U1.21 (IO13)
- new net OUT_NPN0: U1.31 (IO38)
- new net OUT_NPN1: U1.32 (IO39)
- new net OUT_NPN2: U1.33 (IO40)
- new net OUT_NPN3: U1.34 (IO41)
- new net OUT_PNP0: U1.16 (IO46)
- new net OUT_PNP1: U1.24 (IO47)
- new net OUT_RLY1: U1.35 (IO42)
- new net OUT_RLY2: U1.26 (IO45)
- new net RS485_COM: U1.18 (IO10)
- new net RS485_RT: U1.17 (IO9)
- new net RS485_RX: U1.12 (IO8)
- new net TEMP_CS: U1.25 (IO48)
- new net USB+: U1.14 (USB_D+)
- new net USB-: U1.13 (USB_D-)
- no-connect marks 0 -> 5
Other:
- added sheet ENERGY-METER (ENERGY-METER.kicad_sch)
- added sheet IN-0-10V (IN-0-10V.kicad_sch)
- added sheet IN-0-10V1 (IN-0-10V.kicad_sch)
- added sheet IN-4-20mA (IN-4-20mA.kicad_sch)
- added sheet IN-4-20mA1 (IN-4-20mA.kicad_sch)
- added sheet IN-NPN (IN-NPN.kicad_sch)
- added sheet IN-NPN1 (IN-NPN.kicad_sch)
- added sheet IN-NPN2 (IN-NPN.kicad_sch)
- added sheet IN-NPN3 (IN-NPN.kicad_sch)
- added sheet IN-PNP (IN-PNP.kicad_sch)
- added sheet IN-PNP1 (IN-PNP.kicad_sch)
- added sheet OUT-0-10V (OUT-0-10V.kicad_sch)
- added sheet OUT-4-20mA (OUT-4-20mA.kicad_sch)
- added sheet OUT-PNP (OUT-PNP.kicad_sch)
- added sheet RLY (RLY.kicad_sch)
- added sheet TC (TC.kicad_sch)
